File: Schematics/ClockModule.kicad_sch (KiCad schematic)
At the start: 19 parts, among them SW1 SW_Push, SW2 SW_Push_SPDT, U1 NA555P, U2 NA555P, U3 NA555P, U4 74LS06N, U5 74LS08, U6 74LS32

Commit message: Add more data sheets and fix error in clock module schematic
Parts:
- R3: value 1M Ω -> 1K Ω
Changed lines of the file:
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@@
       (effects (font (size 1.27 1.27)) (justify left))
     )
-    (property "Value" "1M Ω" (at 134.62 39.37 0)
+    (property "Value" "1K Ω" (at 134.62 39.37 0)
       (effects (font (size 1.27 1.27)) (justify left))
     )
